File: tester/tester.kicad_pcb (KiCad board)
At the start: 2 copper layers, 184 parts, among them J0 24V, J1 Conn_01x05, J2 BYTE_0, J3 BYTE_1, J4 Conn_02x10_Odd_Even, J5 Conn_01x04_Male, J6 BYTE_0 DO8, J7 BYTE_1 DO8, Q0 BC807, Q1 BC807, Q10 BC807, Q11 BC807, Q12 BC807, Q13 BC807, Q14 BC807, Q15 BC807, Q2 BC807, Q3 BC807, Q4 BC807, Q5 BC807, Q6 BC807, Q7 BC807, Q8 BC807, Q9 BC807, SW0 SW_Push, SW1 SW_Push, SW10 SW_Push, SW11 SW_Push, SW12 SW_Push, SW13 SW_Push, SW14 SW_Push, SW15 SW_Push, SW16 SW_Push, SW2 SW_Push, SW3 SW_Push, SW4 SW_Push, SW5 SW_Push, SW6 SW_Push, SW7 SW_Push, SW8 SW_Push, SW9 SW_Push, U0 LM2596S-ADJ, U1 STM32F103RCTx, U2 ULN2003, U3 ULN2003, U4 ULN2003, Y0 Crystal_Small

Commit message: Finish
First finish
Parts:
- U2, U3, U4: moved to F.Cu
- moved U2 78.6 mm to (71.1, 172.5), turned to 0 degrees
- moved U4 66.6 mm to (71.2, 161.6), turned to 0 degrees
- moved U3 56.0 mm to (71.0, 150.0), turned to 0 degrees
- moved J4 22.3 mm to (119.0, 137.9), turned to 180 degrees
- moved Q14 10.5 mm to (87.4, 197.8)
- moved Q4 10.5 mm to (87.4, 144.8)
- moved Q9 10.5 mm to (87.4, 171.3)
- moved R50 10.5 mm to (81.6, 202.3)
- moved R56 10.5 mm to (81.6, 149.3)
- moved R61 10.5 mm to (81.6, 175.8)
- moved R74 10.5 mm to (84.6, 160.8)
- moved R79 10.5 mm to (84.6, 187.3)
- moved Q1 10.5 mm to (87.4, 128.9)
- moved R53 10.5 mm to (81.6, 133.4)
- moved R67 10.5 mm to (84.6, 123.7)
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Routing:
- net +24V: track 56.5 -> 602.3 mm, vias 0 -> 16
- net GNDD: track 177.5 -> 557.8 mm, vias 2 -> 8
- net VPP: track 24.1 -> 383.5 mm, vias 0 -> 6
- net Net-(D11-Pad1): track 0.00 -> 170.6 mm
- net /16: track 0.00 -> 160.8 mm, vias 0 -> 2
- net /15: track 0.00 -> 154.2 mm, vias 0 -> 2
- net /14: track 0.00 -> 143.9 mm, vias 0 -> 2
- net /13: track 0.00 -> 133.6 mm, vias 0 -> 2
- net /12: track 0.00 -> 124.8 mm, vias 0 -> 2
- net /11: track 0.00 -> 113.1 mm, vias 0 -> 2
- net /10: track 0.00 -> 109.3 mm, vias 0 -> 2
- net Net-(D3-Pad2): track 0.00 -> 108.7 mm, vias 0 -> 1
- net Net-(D18-Pad2): track 0.00 -> 107.9 mm, vias 0 -> 1
- net /8: track 0.00 -> 106.0 mm, vias 0 -> 1
- net /9: track 0.00 -> 105.5 mm, vias 0 -> 2
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- added copper zone on B.Cu, net GNDD
- added copper zone on F.Cu, net GNDD
- added copper zone on B.Cu, net VPP
Other:
- board text added: "+"
- board text added: "+ IN Retom"
- board text added: "+OUT"
- board text added: "-"
- board text added: "-IN Retom"
- board text added: "-OUT"
- board text added: "24 v"
- board text added: "Byte 0"
- board text added: "Byte 1"
- board text added: "Curent"
- board text added: "GND"
- board text added: "Voltage"
